File: ignition_adafruit_ft232h_rD_adapter.kicad_pcb (KiCad board)
At the start: 4 copper layers, 48.3 x 22.9 mm, 12 parts, among them J1 ADAFRUIT_FT232H_REV_D, J2 IGNITION_TARGET_HDR

Commit message: Fixes #1, Fixes #3
Parts:
- removed FID2: iCE40 Adapter, grumpy:Oxide_Board_Identifier_23x6mm
- added Ref**: Val**, tps:OXIDE_Wordmark, B.Cu at (138.0, 90.9)

Commit message: Fixes #5, Fixes #4
Parts:
- moved Ref** 0.14 mm to (138.1, 91.0)
Routing:
- net /CDONE: track 40.3 -> 29.6 mm
- net /~{CRESET}: track 18.5 -> 15.4 mm
- net /~{SPI_SS}: track 30.1 -> 33.1 mm
- net /VCC: track 39.4 -> 41.4 mm
Other:
- board text added: "Ignition Target Programming Adapter for Adafruit FT232H"
- board text removed: "Ignition Target Programming Adapter for Adafruit FT232H rev D"
